File: health_watchy_esp32_c6/power.kicad_sch (KiCad schematic)
At the start: 54 parts, among them J2 JST_2mm_LiPo, J3 TYPE-C-31-M-12, J4 Qwiic_RA, J5 Screw_Terminal_3.5mm_2, J6 Screw_Terminal_3.5mm_2, SW1 SSSS820101, U10 LSM6DS3TR-C, U11 DRV2605LDGS, U5 BQ27441DRZR-G1A, U6 USBLC6-2SC6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

Commit message: Design files update
Parts:
- removed 1V8_TP2: 0.5mm, TestPoint:TestPoint_Pad_1.0x1.0mm, symbol SparkFun-Connector:TestPoint_0.5mm
- removed C2, C20, C32: 10uF, SparkFun-Capacitor:C_0402_1005Metric, symbol SparkFun-Capacitor:10uF_0402_6.3V_20%
- removed C31: 0.1uF, SparkFun-Capacitor:C_0402_1005Metric, symbol SparkFun-Capacitor:0.1uF_0402_16V_10%
- removed C33: 1.0uF, SparkFun-Capacitor:C_0402_1005Metric, symbol SparkFun-Capacitor:1.0uF_0402_16V_10%
- removed J4: Qwiic_RA, SparkFun-Connector:JST_1x04_P1.0mm_Horizontal_SMD, symbol SparkFun-Connector:Qwiic_Right_Angle
- removed J5, J6: Screw_Terminal_3.5mm_2, SparkFun-Connector:ScrewTerminal_1x02_P3.5mm_Horizontal_Black, symbol SparkFun-Connector:Screw_Terminal_3.5mm_2-Black
- removed JP1: Jumper_3_Open, SparkFun-Jumper:Jumper_3_NO, symbol Jumper:Jumper_3_Open
- removed R22, R23: 5.1k, SparkFun-Resistor:R_0402_1005Metric, symbol SparkFun-Resistor:5.1k_0402
- removed U10: LSM6DS3TR-C, LSM6DS3TR-C:LGA-14-2.5X3MM, symbol LSM6DS3TR-C:LSM6DS3TR-C
- removed U11: DRV2605LDGS, Package_SO:VSSOP-10_3x3mm_P0.5mm, symbol Driver_Haptic:DRV2605LDGS
- removed U9: DRV8830DRCR, DRV8830:IC_DRV8830DRCR, symbol DRV8830:DRV8830DRCR
Connections:
- no-connect marks 9 -> 6
Other:
- note removed: "Address: 0x60"
