File: health_watchy_esp32_c6/health_watchy_esp32_c6.kicad_sch (KiCad schematic)
At the start: 1 part, among them U1 ESP32-C6-MINI-1

Commit message: Design files update
Parts:
- added C32: 22uF, SparkFun-Capacitor:C_0402_1005Metric, symbol SparkFun-Capacitor:0.22uF_0402_10V_10%
- added C34, C35, C36, C37, C38: 0.1uF, Capacitor_SMD:C_0402_1005Metric, symbol SparkFun-Capacitor:0.1uF_0402_16V_10%
- added D4: Red, PCM_SparkFun-LED:LED_0402_1005Metric_Red, symbol SparkFun-LED:LED_Red_0402
- added R4, R7: 10k, PCM_SparkFun-Resistor:R_0402_1005Metric, symbol SparkFun-Resistor:10k_0402
- added R5, R6: 0, PCM_SparkFun-Resistor:R_0402_1005Metric, symbol SparkFun-Resistor:0_0402
- added R8: 100, PCM_SparkFun-Resistor:R_0402_1005Metric, symbol SparkFun-Resistor:100_0402
- added SW2, SW3: SMD_4.6x2.8mm_h2.5mm, SparkFun-Switch:Push_SMD_4.6x2.8mm_h2.5mm, symbol SparkFun-Switch:SPST_Push_SMD_4.6x2.8mm_h2.5mm
Connections:
- net GND: now reaches U1.1 (GND), U1.11 (GND), U1.14 (GND), U1.2 (GND), U1.36 (GND), U1.37 (GND), U1.38 (GND), U1.39 (GND), U1.40 (GND), U1.41 (GND), U1.42 (GND), U1.43 (GND), U1.44 (GND), U1.45 (GND), U1.46 (GND), U1.47 (GND), U1.48 (GND), U1.49 (GND), U1.50 (GND), U1.51 (GND), U1.52 (GND), U1.53 (GND)
- net GND: now also C32.2, C34.2, C35.2, C36.2, C37.2, C38.1, D4.1 (K), SW2.1, SW3.1
- net Sensor Sheet/HAPT_IN: now reaches U1.10 (IO5)
- net Sensor Sheet/HAPT_EN: now reaches U1.15 (IO6)
- net USB.FILT.D-: now reaches U1.17 (IO12)
- net USB.FILT.D-: now also R5.1
- net USB.FILT.D+: now reaches U1.18 (IO13)
- net USB.FILT.D+: now also R6.1
- net IO8: now reaches U1.22 (IO8)
- net IO8: now also R7.1
- net ~{BOOT}: now reaches U1.23 (IO9)
- net ~{BOOT}: now also SW3.2
- net SCL: now reaches U1.24 (IO18)
- net SDA: now reaches U1.25 (IO19)
- net Power Subsystem/BQ27441.GPOUT: now reaches U1.26 (IO20)
- net Power Subsystem/~{BQ24075.CHG}: now reaches U1.27 (IO21)
- net Power Subsystem/~{BQ24075.PGOOD}: now reaches U1.28 (IO22)
- net Power Subsystem/BQ27441.BIN: now reaches U1.29 (IO23)
- net +3.3V: now reaches U1.3 (3V3)
- net +3.3V: now also C32.1, C34.1, R4.2, R7.2
- net at U1.6 (IO3): now also R8.2
- net ~{RESET}: now reaches U1.8 (EN)
- net ~{RESET}: now also C35.1, C38.2, R4.1, SW2.2
- net Sensor Sheet/LSM6_INT1: now reaches U1.9 (IO4)
- new net: D4.2 (A), R8.1
- new net Power Subsystem/USB.D+: C36.1, R6.2
- new net Power Subsystem/USB.D-: C37.1, R5.2
Other:
- added sheet Sensor Sheet (sensor_sheet.kicad_sch)
- sheet Power Subsystem ports: added BQ27441.BIN, BQ27441.GPOUT, SCL, SDA, USB.D+, USB.D-, ~{BQ24075.CHG}, ~{BQ24075.PGOOD}; removed none
- moved on the sheet: U1

Commit message: Checking in library
Parts:
- added C39, C40: 12pF, PCM_SparkFun-Capacitor:C_0402_1005Metric, symbol SparkFun-Capacitor:12pF_0402_50V_5%
- added R10, R11, R12, R9: 100k, PCM_SparkFun-Resistor:R_0402_1005Metric, symbol SparkFun-Resistor:100k_0402
- added SW4, SW5, SW6, SW7: ~, K2-1114SA-A4SW-06:KEY-SMD_4P-L4.8-W4.6-P1.70-LS6.2, symbol K2-1114SA-A4SW-06:K2-1114SA-A4SW-06
- added TP1, TP2: 0.5mm, PCM_SparkFun-Connector:TestPoint-0.5mm, symbol SparkFun-Connector:TestPoint_0.5mm
- added U9: ~, Sr2HARU:UDFN-6_L1.6-W1.3-P0.40-TL, symbol Sr2HARU:SR2HARU
- added Y2: 32.768kHz, PCM_SparkFun-Clock:Crystal_SMD_3.2x1.5mm, symbol SparkFun-Clock:Crystal_32.768kHz_3.2x1.5mm
Connections:
- net +3.3V: now also R10.2, R11.2, R12.2, R9.2, U9.6 (VCC)
- net GND: now also C39.1, C40.1, SW4.3, SW4.4, SW5.3, SW5.4, SW6.3, SW6.4, SW7.3, SW7.4, U9.1 (VSS)
- net ~{RESET}: now also U9.3 (RST#)
- net CLK.IN: now reaches U1.12 (IO0)
- net CLK.IN: now also C39.2, Y2.2
- net CLK.OUT: now reaches U1.13 (IO1)
- net CLK.OUT: now also C40.2, Y2.1
- net BTN3: now reaches U1.16 (IO7)
- net BTN3: now also R11.1, SW6.1, SW6.2, U9.5 (SR0#)
- net BTN4: now reaches U1.19 (IO14)
- net BTN4: now also R12.1, SW7.1, SW7.2
- net BTN2: now reaches U1.20 (IO15)
- net BTN2: now also R10.1, SW5.1, SW5.2, U9.2 (SR1#)
- net RXD0: now reaches U1.30 (RXD0)
- net RXD0: now also TP2.1
- net TXD0: now reaches U1.31 (TXD0)
- net TXD0: now also TP1.1
- net BTN1: now reaches U1.5 (IO2)
- net BTN1: now also R9.1, SW4.1, SW4.2
- no-connect marks 0 -> 1
Other:
- sheet Sensor Sheet ports: added BUSY, CS, DC, GDR, MOSI, PREVGH, PREVGL, RES, RESE, SCK, ~{INT_RTC}, ~{MAX30205_OS}; removed none
- moved on the sheet: D4, R8

Commit message: Checking in completed design files.
Parts:
- removed C36, C37: 0.1uF, Capacitor_SMD:C_0402_1005Metric, symbol SparkFun-Capacitor:0.1uF_0402_16V_10%
- removed C39, C40: 12pF, PCM_SparkFun-Capacitor:C_0402_1005Metric, symbol SparkFun-Capacitor:12pF_0402_50V_5%
- removed R5, R6: 0, PCM_SparkFun-Resistor:R_0402_1005Metric, symbol SparkFun-Resistor:0_0402
- removed Y2: 32.768kHz, PCM_SparkFun-Clock:Crystal_SMD_3.2x1.5mm, symbol SparkFun-Clock:Crystal_32.768kHz_3.2x1.5mm
- added C2, C20, C22, C23: 10uF, SparkFun-Capacitor:C_0402_1005Metric, symbol SparkFun-Capacitor:10uF_0402_6.3V_20%
- added C24, C25: 0.1uF, SparkFun-Capacitor:C_0402_1005Metric, symbol SparkFun-Capacitor:0.1uF_0402_16V_10%
- added D5: MBR0530, SparkFun-Semiconductor-Standard:SOD-523, symbol Diode:MBR0530
- added D6: Yellow, LED_SMD:LED_0402_1005Metric, symbol SparkFun-LED:LED_Yellow_0402
- added D7: Green, LED_SMD:LED_0402_1005Metric, symbol SparkFun-LED:LED_Yellow_0402
- added J2: 532610271, 532610271:MOLEX_532610271, symbol 532610271:532610271
- added J5: USB_B_Micro, Connector_USB:USB_Micro-B_Amphenol_10103594-0001LF_Horizontal, symbol Connector:USB_B_Micro
- added L2: 2.2nH, Inductor_SMD:L_0402_1005Metric, symbol SparkFun-Coil:2.2nH_0603_0.5A
- added Q2: AO3401A, Package_TO_SOT_SMD:SOT-23, symbol Transistor_FET:AO3401A
- added R13, R15: 10k, Resistor_SMD:R_0402_1005Metric, symbol SparkFun-Resistor:10k_0402
- added R14: 1k, Resistor_SMD:R_0402_1005Metric, symbol SparkFun-Resistor:1k_0402
- added R16, R17: 100k, Resistor_SMD:R_0402_1005Metric, symbol SparkFun-Resistor:100k_0402
- added U5: ME6211C33M5, Package_TO_SOT_SMD:SOT-23-5, symbol Regulator_Linear:ME6211C33M5
- added U6: TP4057, Package_TO_SOT_SMD:TSOT-23-6, symbol Battery_Management:TP4057
- D4: footprint PCM_SparkFun-LED:LED_0402_1005Metric_Red -> SparkFun-LED:LED_0402_1005Metric_Red
- R10, R11, R12, R4, R7, R8, R9: footprint PCM_SparkFun-Resistor:R_0402_1005Metric -> SparkFun-Resistor:R_0402_1005Metric
- TP1, TP2: footprint PCM_SparkFun-Connector:TestPoint-0.5mm -> SparkFun-Connector:TestPoint-0.5mm
- U9: footprint Sr2HARU:UDFN-6_L1.6-W1.3-P0.40-TL -> SR2HARU:UDFN-6_L1.6-W1.3-P0.40-TL
Connections:
- net CLK.OUT is gone; now on an unnamed net: U1.13 (IO1)
- net Power Subsystem/BQ27441.BIN is gone; now on net Sensor Sheet/RES: U1.29 (IO23)
- net Power Subsystem/BQ27441.GPOUT is gone; now on net BTN1: U1.26 (IO20)
- net Power Subsystem/~{BQ24075.PGOOD} is gone; now on net Sensor Sheet/BUSY: U1.28 (IO22)
- net Sensor Sheet/HAPT_EN is gone; now on net Sensor Sheet/DC: U1.15 (IO6)
- net Sensor Sheet/HAPT_IN is gone; now on net Sensor Sheet/MOSI: U1.10 (IO5)
- net Sensor Sheet/LSM6_INT1 is gone; now on net Sensor Sheet/SCK: U1.9 (IO4)
- net +3.3V: now also C2.1, U5.5 (V_{OUT})
- net BTN1: no longer U1.5 (IO2)
- net BTN2: no longer SW5.2
- net BTN3: now also U1.5 (IO2); no longer SW6.1, U1.16 (IO7)
- net GND: now also C2.2, C20.2, C22.2, C23.1, C24.2, C25.2, J2.2, J2.S1 (SHIELD1), J2.S2 (SHIELD2), J5.5 (GND), J5.6 (Shield), R13.1, R15.1, R17.1, U5.2 (V_{SS}), U6.2 (GND); no longer SW5.4, SW6.3
- net Sensor Sheet/CS: now also U1.16 (IO7)
- net at R8.2: no longer U1.6 (IO3)
- net CLK.IN renamed ADC
- net ADC: now also R16.1, R17.2
- net Power Subsystem/~{BQ24075.CHG}: no longer names the net of U1.27 (IO21)
- net USB.FILT.D+ renamed USB.D+
- net USB.D+: now also J5.3 (D+)
- net USB.FILT.D- renamed USB.D-
- net USB.D-: now also J5.2 (D-)
- new net: D6.2 (A), D7.2 (A), R14.1
- new net: D7.1 (K), U6.5 (STDBY)
- new net: D6.1 (K), U6.1 (~{CHRG})
- new net +BATT: C23.2, J2.1, Q2.3 (D), R16.2, U6.3 (BAT)
- new net 5V: C25.1, J5.1 (VBUS), L2.2
- new net PROG: R15.2, U6.6 (PROG)
- new net VIN: C20.1, D5.1 (K), Q2.2 (S), U5.1 (V_{IN}), U5.3 (CE)
- new net VUSB: C22.1, C24.1, D5.2 (A), L2.1, Q2.1 (G), R13.2, R14.2, U6.4 (V_{CC})
- no-connect marks 1 -> 8
Other:
- removed sheet Power Subsystem
- sheet Sensor Sheet ports: added none; removed GDR, HAPT_EN, HAPT_IN, LSM6_INT1, PREVGH, PREVGL, RESE, ~{INT_RTC}, ~{MAX30205_OS}
- moved on the sheet: D4, R11, R8
