File: health_watchy_esp32_c6/sensor_sheet.kicad_sch (KiCad schematic)
At the start: 45 parts, among them J1 Conn_01x24_FPC, J4 Qwiic_RA, J6 Screw_Terminal_3.5mm_2, Q1 AO3404A, U10 LSM6DS3TR-C, U11 DRV2605LDGS, U12 AP2127-1.8, U2 PCF8563T, U3 MAX30205MTA, U4 MAX30102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

Commit message: Checking in library
Parts:
- added U13: ~, PCA9500:HVQFN-16_L4.0-W4.0-P0.65-TL-EP2.2, symbol PCA9500:PCA9500BS,118
- C17, C18: footprint PCM_SparkFun-Capacitor:C_0402_1005Metric -> SparkFun-Capacitor:C_0402_1005Metric
Changed lines of the file:
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@@
 			)
 		)
-		(property "Footprint" "PCM_SparkFun-Capacitor:C_0402_1005Metric"
+		(property "Footprint" "SparkFun-Capacitor:C_0402_1005Metric"
 			(at 186.69 135.89 0)
 			(effects
@@
 			)
 		)
-		(property "Footprint" "PCM_SparkFun-Capacitor:C_0402_1005Metric"
+		(property "Footprint" "SparkFun-Capacitor:C_0402_1005Metric"
 			(at 172.72 147.32 0)
 			(effects
@@
 					(unit 1)
 				)
+			)
+		)
+	)
+	(symbol
+		(lib_id "PCA9500:PCA9500BS,118")
+		(at 238.76 123.19 0)
+		(unit 1)
+		(exclude_from_sim no)
+		(in_bom yes)
+		(on_board yes)
+		(dnp no)
+		(fields_autoplaced yes)
+		(property "Reference" "U13"
+			(at 238.125 138.43 0)
+			(effects
+				(font
+					(size 1.27 1.27)
+				)
+			)
+		)
+		(property "Value" "~"
+			(at 238.125 140.97 0)
+			(effects
+				(font
+					(size 1.27 1.27)
+				)
+			)
+		)
+		(property "Footprint" "PCA9500:HVQFN-16_L4.0-W4.0-P0.65-TL-EP2.2"
+			(at 238.76 123.19 0)
+			(effects
+				(font
+					(size 1.27 1.27)
+				)
+				(hide yes)
+			)
+		)
+		(property "Datasheet" "https://www.nxp.com/docs/en/data-sheet/PCA9500.pdf"
+			(at 238.76 123.19 0)
+			(effects
+				(font
+					(size 1.27 1.27)
+				)
+				(hide yes)
+			)
+		)
+		(property "Description" "Interface:- Interrupt Output:- Output Type:-"
+			(at 238.76 123.19 0)
+			(effects
+				(font
+					(size 1.27 1.27)
+				)
+				(hide yes)
+			)
+		)
+		(property "Manufacturer Part" "PCA9500BS,118"
+			(at 238.76 123.19 0)
+			(effects
+				(font
+					(size 1.27 1.27)
+				)
+				(hide yes)
+			)
+		)
+		(property "Manufacturer" "NXP(恩智浦)"
+			(at 238.76 123.19 0)
+			(effects
+				(font
+					(size 1.27 1.27)
+				)
+				(hide yes)
+			)
+		)
+		(property "Supplier Part" "C2669724"
+			(at 238.76 123.19 0)
+			(effects
+				(font
+					(size 1.27 1.27)
+				)
+				(hide yes)
+			)
+		)
+		(property "Supplier" "LCSC"
+			(at 238.76 123.19 0)
+			(effects
+				(font
+					(size 1.27 1.27)
+				)
+				(hide yes)
+			)
+		)
+		(property "LCSC Part Name" "PCA9500BS,118"
+			(at 238.76 123.19 0)
+			(effects
+				(font
+					(size 1.27 1.27)
+				)
+				(hide yes)
+			)
+		)
+		(pin "13"
+		)
+		(pin "11"
+		)
+		(pin "2"
+		)
+		(pin "3"
+		)
+		(pin "10"
+		)
+		(pin "8"
+		)
+		(pin "15"
+		)
+		(pin "12"
+		)
+		(pin "5"
+		)
+		(pin "9"
+		)
+		(pin "4"
+		)
+		(pin "1"
+		)
+		(pin "6"
+		)
+		(pin "7"
+		)
+		(pin "16"
+		)
+		(pin "17"
+		)
+		(pin "14"
+		)
+		(instances
+			(project ""
+				(path "/16ba0087-9056-428c-a819-683762e5f891/d331b73b-4395-4ceb-b0c5-eb302da6d8a8"
+					(reference "U13")
+					(unit 1)
+				)

Commit message: Checking in completed design files.
Parts:
- removed 1V8_TP2: 0.5mm, TestPoint:TestPoint_Pad_1.0x1.0mm, symbol SparkFun-Connector:TestPoint_0.5mm
- removed C1, C2, C20, C8: 10uF, SparkFun-Capacitor:C_0402_1005Metric, symbol SparkFun-Capacitor:10uF_0402_6.3V_20%
- removed C3, C4: 15pF, SparkFun-Capacitor:C_0402_1005Metric, symbol SparkFun-Capacitor:15pF_0402_50V_5%
- removed C33: 1.0uF, SparkFun-Capacitor:C_0402_1005Metric, symbol SparkFun-Capacitor:1.0uF_0402_16V_10%
- removed J4: Qwiic_RA, SparkFun-Connector:JST_1x04_P1.0mm_Horizontal_SMD, symbol SparkFun-Connector:Qwiic_Right_Angle
- removed J6: Screw_Terminal_3.5mm_2, SparkFun-Connector:ScrewTerminal_1x02_P3.5mm_Horizontal_Black, symbol SparkFun-Connector:Screw_Terminal_3.5mm_2-Black
- removed JP1: Jumper_3_Open, SparkFun-Jumper:Jumper_3_NO, symbol Jumper:Jumper_3_Open
- removed Q1: AO3404A, Package_TO_SOT_SMD:SOT-223-3_TabPin2, symbol SparkFun-DiscreteSemi:Q_NMOS_5.8A_30V
- removed U11: DRV2605LDGS, Package_SO:VSSOP-10_3x3mm_P0.5mm, symbol Driver_Haptic:DRV2605LDGS
- removed U13: ~, PCA9500:HVQFN-16_L4.0-W4.0-P0.65-TL-EP2.2, symbol PCA9500:PCA9500BS,118
- removed U2: PCF8563T, Package_SO:SOIC-8_3.9x4.9mm_P1.27mm, symbol Timer_RTC:PCF8563T
- removed Y1: 32.768kHz, Crystal:Crystal_SMD_G8-2Pin_3.2x1.5mm, symbol SparkFun-Clock:Crystal_32.768kHz_3.2x1.5mm
- added C1: 0.1uF, SparkFun-Capacitor:C_0402_1005Metric, symbol SparkFun-Capacitor:0.1uF_0402_16V_10%
- added Q4: AO3400A, Package_TO_SOT_SMD:SOT-23, symbol Transistor_FET:AO3400A
- added U2: RV-8803-C7-32.768KHZ-3PPM-TA-QC, RV-8803-C7-32.768KHZ-3PPM-TA-QC:IC_RV-8803-C7-32.768KHZ-3PPM-TA-QC, symbol RV-8803-C7-32.768KHZ-3PPM-TA-QC:RV-8803-C7-32.768KHZ-3PPM-TA-QC
- D1, D2, D3: footprint Diode_SMD:D_SOD-123 -> Diode_SMD:D_SOD-523
- J1: footprint PCM_SparkFun-Connector:FPC_1x24_P0.5mm_Horizontal_BottomContact -> SparkFun-Connector:FPC_1x24_P0.5mm_Horizontal_BottomContact
- R1, R3: footprint PCM_SparkFun-Resistor:R_0402_1005Metric -> SparkFun-Resistor:R_0402_1005Metric
- U12: footprint PCM_SparkFun-Semiconductor-Standard:SOT23-5 -> SparkFun-Semiconductor-Standard:SOT23-5
Connections:
- net JMP.SCL is gone; now on net +3.3V: R23.2
- net JMP.SDA is gone; now on net +3.3V: R22.2
- net VOUT is gone; now on net +3.3V: C5.2, U3.8 (VDD)
- net +3.3V: now also C7.1, U12.1 (VIN), U12.3 (EN), C1.1, U2.3 (VDD)
- net 3.3V: no longer C7.1, U12.1 (VIN)
- net GDR: now also Q4.1 (G)
- net GND: now also C1.2, U2.5 (VSS)
- net RESE: now also Q4.2 (S)
- net SCL: now also U2.8 (SCL)
- net SDA: now also U2.1 (SDA)
- net at C18.2, D1.2 (A), L1.2: now also Q4.3 (D)
- net LSM6_INT1: no longer names the net of U10.4 (INT1)
- net ~{INT_MAX30102}: no longer names the net of U4.13 (~{INT})
- net ~{MAX30205_OS}: no longer names the net of U3.3 (OS)
- no-connect marks 7 -> 14
Other:
- moved on the sheet: R22, R23, R3
